File: KiCad/Projects/GenLOCK Drone/NRF905.sch (KiCad schematic (older format))
At the start: 3 parts, among them U1 NRF905

Commit message: .
Parts:
- added AE?: Antenna, symbol Device:Antenna
- added C?: 3.3nF, symbol Device:C_Small
- added C? (x2): 0F, symbol Device:C_Small
- added C? (x2): 18PF, symbol Device:C_Small
- added C?: 180PF, symbol Device:C_Small
- added C?: 6.8PF, symbol Device:C_Small
- added L?: 12nH, symbol pspice:INDUCTOR
- added L? (x2): 39nH, symbol pspice:INDUCTOR
Connections:
- net GNDREF: now also C?.1, C?.1, C?.2, C?.2, C?.2
- net at U1.19 (VDD_PA): now also C?.1, C?.2, L?.1
- net at U1.20 (ANT1): now also C?.1, C?.2, L?.1, L?.2
- net at U1.21 (ANT2): now also C?.1, C?.2, L?.2, L?.2
- new net: C?.1, L?.1
- new net: AE?.1 (A), C?.1, C?.2
Changed lines of the file:
@@
 EESchema Schematic File Version 4
+LIBS:GenLOCK Drone-cache
 EELAYER 29 0
 EELAYER END
@@
 	0    -1   -1   0
 $EndComp
+Wire Wire Line
+	5300 3800 5150 3800
+Wire Wire Line
+	5150 3800 5150 3750
+Wire Wire Line
+	5150 3750 4350 3750
+Wire Wire Line
+	4350 3750 4350 4250
+Wire Wire Line
+	4350 4250 4500 4250
+$Comp
+L Device:C_Small C?
+U 1 1 5CED52A1
+P 4600 4250
+F 0 "C?" V 4700 4250 50  0000 C CNN
+F 1 "3.3nF" V 4500 4250 50  0000 C CNN
+F 2 "" H 4600 4250 50  0001 C CNN
+F 3 "~" H 4600 4250 50  0001 C CNN
+	1    4600 4250
+	0    1    1    0
+$EndComp
+$Comp
+L power:GNDREF #PWR?
+U 1 1 5CED5DBC
+P 4700 4250
+F 0 "#PWR?" H 4700 4000 50  0001 C CNN
+F 1 "GNDREF" V 4705 4122 50  0000 R CNN
+F 2 "" H 4700 4250 50  0001 C CNN
+F 3 "" H 4700 4250 50  0001 C CNN
+	1    4700 4250
+	0    -1   -1   0
+$EndComp
+Wire Wire Line
+	4850 2150 4850 2450
+Wire Wire Line
+	3950 2450 3950 2350
+Wire Wire Line
+	3950 1750 4400 1750
+Wire Wire Line
+	4850 2050 5300 2050
+Wire Wire Line
+	4850 2150 5300 2150
+Wire Wire Line
+	3950 2450 4400 2450
+Wire Wire Line
+	4850 1750 4850 2050
+$Comp
+L Device:C_Small C?
+U 1 1 5CED9A7D
+P 4400 2100
+F 0 "C?" H 4492 2146 50  0000 L CNN
+F 1 "0F" H 4492 2055 50  0000 L CNN
+F 2 "" H 4400 2100 50  0001 C CNN
+F 3 "~" H 4400 2100 50  0001 C CNN
+	1    4400 2100
+	1    0    0    -1
+$EndComp
+Wire Wire Line
+	4400 2000 4400 1750
+Connection ~ 4400 1750
+Wire Wire Line
+	4400 1750 4850 1750
+Wire Wire Line
+	4400 2200 4400 2450
+Connection ~ 4400 2450
+Wire Wire Line
+	4400 2450 4850 2450
+$Comp
+L Device:C_Small C?
+U 1 1 5CEDBFEF
+P 4400 2550
+F 0 "C?" H 4492 2596 50  0000 L CNN
+F 1 "18PF" H 4492 2505 50  0000 L CNN
+F 2 "" H 4400 2550 50  0001 C CNN
+F 3 "~" H 4400 2550 50  0001 C CNN
+	1    4400 2550
+	1    0    0    -1
+$EndComp
+$Comp
+L Device:C_Small C?
+U 1 1 5CEDC357
+P 4400 1650
+F 0 "C?" H 4492 1696 50  0000 L CNN
+F 1 "18PF" H 4492 1605 50  0000 L CNN
+F 2 "" H 4400 1650 50  0001 C CNN
+F 3 "~" H 4400 1650 50  0001 C CNN
+	1    4400 1650
+	1    0    0    -1
+$EndComp
+$Comp
+L power:GNDREF #PWR?
+U 1 1 5CEDC733
+P 4400 2650
+F 0 "#PWR?" H 4400 2400 50  0001 C CNN
+F 1 "GNDREF" H 4405 2477 50  0000 C CNN
+F 2 "" H 4400 2650 50  0001 C CNN
+F 3 "" H 4400 2650 50  0001 C CNN
+	1    4400 2650
+	1    0    0    -1
+$EndComp
+$Comp
+L power:GNDREF #PWR?
+U 1 1 5CEDC9CC
+P 4400 1550
+F 0 "#PWR?" H 4400 1300 50  0001 C CNN
+F 1 "GNDREF" H 4405 1377 50  0000 C CNN
+F 2 "" H 4400 1550 50  0001 C CNN
+F 3 "" H 4400 1550 50  0001 C CNN
+	1    4400 1550
+	-1   0    0    1
+$EndComp
+$Comp
+L pspice:INDUCTOR L?
+U 1 1 5CEDCDC7
+P 3950 2100
+F 0 "L?" V 3904 2178 50  0000 L CNN
+F 1 "12nH" V 3995 2178 50  0000 L CNN
+F 2 "" H 3950 2100 50  0001 C CNN
+F 3 "~" H 3950 2100 50  0001 C CNN
+	1    3950 2100
+	0    1    1    0
+$EndComp
+Wire Wire Line
+	3950 1850 3950 1750
+Wire Wire Line
+	3950 1750 3850 1750
+Connection ~ 3950 1750
+$Comp
+L pspice:INDUCTOR L?
+U 1 1 5CEDE77F
+P 3600 1750
+F 0 "L?" H 3450 1850 50  0000 C CNN
+F 1 "39nH" H 3700 1850 50  0000 C CNN
+F 2 "" H 3600 1750 50  0001 C CNN
+F 3 "~" H 3600 1750 50  0001 C CNN
+	1    3600 1750
+	1    0    0    -1
+$EndComp
+Wire Wire Line
+	4350 3750 3300 3750
+Wire Wire Line
+	3300 3750 3300 1750
+Wire Wire Line
+	3300 1750 3350 1750
+Connection ~ 4350 3750
+$Comp
+L Device:C_Small C?
+U 1 1 5CEE10EB
+P 3200 1750
+F 0 "C?" V 2971 1750 50  0000 C CNN
+F 1 "180PF" V 3062 1750 50  0000 C CNN
+F 2 "" H 3200 1750 50  0001 C CNN
+F 3 "~" H 3200 1750 50  0001 C CNN
+	1    3200 1750
+	0    1    1    0
+$EndComp
+Connection ~ 3300 1750
+Wire Wire Line
+	3100 1750 3000 1750
+$Comp
+L power:GNDREF #PWR?
+U 1 1 5CEE2B51
+P 3000 1750
+F 0 "#PWR?" H 3000 1500 50  0001 C CNN
+F 1 "GNDREF" V 3005 1622 50  0000 R CNN
+F 2 "" H 3000 1750 50  0001 C CNN
+F 3 "" H 3000 1750 50  0001 C CNN
+	1    3000 1750
+	0    1    1    0
+$EndComp
+$Comp
+L pspice:INDUCTOR L?
+U 1 1 5CEE2D59
+P 3600 2450
+F 0 "L?" H 3450 2550 50  0000 C CNN
+F 1 "39nH" H 3700 2550 50  0000 C CNN
+F 2 "" H 3600 2450 50  0001 C CNN
+F 3 "~" H 3600 2450 50  0001 C CNN
+	1    3600 2450
+	1    0    0    -1
+$EndComp
+Wire Wire Line
+	3850 2450 3950 2450
+Connection ~ 3950 2450
+$Comp
+L Device:C_Small C?
+U 1 1 5CEE5F1E
+P 3150 2450
+F 0 "C?" V 2921 2450 50  0000 C CNN
+F 1 "6.8PF" V 3012 2450 50  0000 C CNN
+F 2 "" H 3150 2450 50  0001 C CNN
+F 3 "~" H 3150 2450 50  0001 C CNN
+	1    3150 2450
+	0    1    1    0
+$EndComp
+Wire Wire Line
+	3250 2450 3350 2450
+Wire Wire Line
+	3050 2450 3000 2450
+Wire Wire Line
+	3000 2450 3000 2500
+Connection ~ 3000 2450
+Wire Wire Line
+	3000 2450 2950 2450
+$Comp
+L Device:C_Small C?
+U 1 1 5CEEA35A
+P 3000 2600
+F 0 "C?" H 3092 2646 50  0000 L CNN
+F 1 "0F" H 3092 2555 50  0000 L CNN
+F 2 "" H 3000 2600 50  0001 C CNN
+F 3 "~" H 3000 2600 50  0001 C CNN
+	1    3000 2600
+	1    0    0    -1
+$EndComp
+$Comp
+L power:GNDREF #PWR?
+U 1 1 5CEEA8A2
+P 3000 2700
+F 0 "#PWR?" H 3000 2450 50  0001 C CNN
+F 1 "GNDREF" H 3005 2527 50  0000 C CNN
+F 2 "" H 3000 2700 50  0001 C CNN
+F 3 "" H 3000 2700 50  0001 C CNN
+	1    3000 2700
+	1    0    0    -1
+$EndComp
+$Comp
+L Device:Antenna AE?
+U 1 1 5CEEB254
+P 2750 2450
+F 0 "AE?" V 2967 2393 50  0000 C CNN
+F 1 "Antenna" V 2876 2393 50  0000 C CNN
+F 2 "" H 2750 2450 50  0001 C CNN
+F 3 "~" H 2750 2450 50  0001 C CNN
+	1    2750 2450
+	0    -1   -1   0
+$EndComp

Commit message: .
Parts:
- added C?: 33PF, symbol Device:C_Small
- added C? (x2): 10PF, symbol Device:C_Small
- added R?: 1M, symbol Device:R_Small_US
- added X?: XO32, Oscillator:Oscillator_SMD_EuroQuartz_XO32-4Pin_3.2x2.5mm, symbol Oscillator:XO32
Connections:
- net +3V3: now also C?.2
- net GNDREF: now also C?.1, C?.1, C?.1, X?.2 (GND), X?.4 (V+)
- net MISO: now reaches U1.10 (MISO)
- net MOSI: now reaches U1.11 (MOSI)
- net SPI_SCK: now reaches U1.12 (SCK)
- net SPI_CSN: now reaches U1.13 (CSN)
- net at U1.14 (xc1): now also C?.2, R?.1, X?.1 (EN)
- net at U1.15 (xc2): now also C?.2, R?.2, X?.3 (OUT)
- net CD: now reaches U1.6 (CD)
- net AM: now reaches U1.7 (AM)
- net DR: now reaches U1.8 (DR)
Other:
- moved on the sheet: C?
Changed lines of the file:
@@
 Text Label 6900 2250 2    50   ~ 0
 uPCLK
-Text HLabel 6900 2250 2    50   Input ~ 0
+Text HLabel 6900 2250 2    50   Output ~ 0
 uPCLK
 Wire Wire Line
@@
 	5150 3750 4350 3750
 Wire Wire Line
-	4350 3750 4350 4250
-Wire Wire Line
-	4350 4250 4500 4250
+	4350 3750 4350 3850
 $Comp
 L Device:C_Small C?
 U 1 1 5CED52A1
-P 4600 4250
-F 0 "C?" V 4700 4250 50  0000 C CNN
-F 1 "3.3nF" V 4500 4250 50  0000 C CNN
-F 2 "" H 4600 4250 50  0001 C CNN
-F 3 "~" H 4600 4250 50  0001 C CNN
-	1    4600 4250
-	0    1    1    0
+P 4350 3950
+F 0 "C?" V 4450 3950 50  0000 C CNN
+F 1 "3.3nF" V 4250 3950 50  0000 C CNN
+F 2 "" H 4350 3950 50  0001 C CNN
+F 3 "~" H 4350 3950 50  0001 C CNN
+	1    4350 3950
+	-1   0    0    1
 $EndComp
 $Comp
 L power:GNDREF #PWR?
 U 1 1 5CED5DBC
-P 4700 4250
-F 0 "#PWR?" H 4700 4000 50  0001 C CNN
-F 1 "GNDREF" V 4705 4122 50  0000 R CNN
-F 2 "" H 4700 4250 50  0001 C CNN
-F 3 "" H 4700 4250 50  0001 C CNN
-	1    4700 4250
-	0    -1   -1   0
+P 4350 4050
+F 0 "#PWR?" H 4350 3800 50  0001 C CNN
+F 1 "GNDREF" V 4355 3922 50  0000 R CNN
+F 2 "" H 4350 4050 50  0001 C CNN
+F 3 "" H 4350 4050 50  0001 C CNN
+	1    4350 4050
+	1    0    0    -1
 $EndComp
 Wire Wire Line
@@
 	0    -1   -1   0
 $EndComp
+Wire Wire Line
+	6600 2350 6900 2350
+Text Label 6900 2350 2    50   ~ 0
+CD
+Text HLabel 6900 2350 2    50   Output ~ 0
+CD
+Wire Wire Line
+	6600 2450 6900 2450
+Text Label 6900 2450 2    50   ~ 0
+AM
+Text HLabel 6900 2450 2    50   Output ~ 0
+AM
+Wire Wire Line
+	6050 4350 6150 4350
+Connection ~ 6050 4350
+$Comp
+L Device:C_Small C?
+U 1 1 5CEDE401
+P 6250 4350
+F 0 "C?" V 6400 4350 50  0000 C CNN
+F 1 "33PF" V 6112 4350 50  0000 C CNN
+F 2 "" H 6250 4350 50  0001 C CNN
+F 3 "~" H 6250 4350 50  0001 C CNN
+	1    6250 4350
+	0    1    1    0
+$EndComp
+$Comp
+L power:GNDREF #PWR?
+U 1 1 5CEDF64B
+P 6350 4350
+F 0 "#PWR?" H 6350 4100 50  0001 C CNN
+F 1 "GNDREF" V 6355 4222 50  0000 R CNN
+F 2 "" H 6350 4350 50  0001 C CNN
+F 3 "" H 6350 4350 50  0001 C CNN
+	1    6350 4350
+	0    -1   -1   0
+$EndComp
+Wire Wire Line
+	6600 2550 6900 2550
+Text Label 6900 2550 2    50   ~ 0
+DR
+Text HLabel 6900 2550 2    50   Output ~ 0
+DR
+Wire Wire Line
+	6600 2700 6900 2700
+Text HLabel 6900 2700 2    50   Output ~ 0
+MISO
+Text Label 6900 2700 2    50   ~ 0
+MISO
+Wire Wire Line
+	6600 2800 6900 2800
+Text HLabel 6900 2800 2    50   Input ~ 0
+MOSI
+Text Label 6900 2800 2    50   ~ 0
+MOSI
+Wire Wire Line
+	6600 2900 6900 2900
+Text Label 6900 2900 2    50   ~ 0
+SPI_SCK
+Wire Wire Line
+	6600 3000 6900 3000
+Text Label 6900 3000 2    50   ~ 0
+SPI_CSN
+Text HLabel 6900 2900 2    50   Input ~ 0
+SPI_SCK
+Text HLabel 6900 3000 2    50   Input ~ 0
+SPI_CSN
+Wire Wire Line
+	6600 3250 6750 3250
+Wire Wire Line
+	6750 3250 6750 3150
+Wire Wire Line
+	6600 3150 6700 3150
+Wire Wire Line
+	6700 3150 6700 3050
+$Comp
+L Oscillator:XO32 X?
+U 1 1 5CEF225C
+P 8300 3100
+F 0 "X?" V 8254 3444 50  0000 L CNN
+F 1 "XO32" V 8345 3444 50  0000 L CNN
+F 2 "Oscillator:Oscillator_SMD_EuroQuartz_XO32-4Pin_3.2x2.5mm" H 9000 2750 50  0001 C CNN
+F 3 "http://cdn-reichelt.de/documents/datenblatt/B400/XO32.pdf" H 8200 3100 50  0001 C CNN
+	1    8300 3100
+	0    1    1    0
+$EndComp
+Wire Wire Line
+	7850 2800 8300 2800
+Wire Wire Line
+	6700 3050 7750 3050
+Wire Wire Line
+	8300 2800 8650 2800
+Connection ~ 8300 2800
+$Comp
+L Device:C_Small C?
+U 1 1 5CEF7465
+P 8750 2800
+F 0 "C?" V 8521 2800 50  0000 C CNN
+F 1 "10PF" V 8612 2800 50  0000 C CNN
+F 2 "" H 8750 2800 50  0001 C CNN
+F 3 "~" H 8750 2800 50  0001 C CNN
+	1    8750 2800
+	0    1    1    0
+$EndComp
+Wire Wire Line
+	8850 2800 8950 2800
+$Comp
+L power:GNDREF #PWR?
+U 1 1 5CEF9ACB
+P 9100 2800
+F 0 "#PWR?" H 9100 2550 50  0001 C CNN
+F 1 "GNDREF" H 9105 2627 50  0000 C CNN
+F 2 "" H 9100 2800 50  0001 C CNN
+F 3 "" H 9100 2800 50  0001 C CNN
+	1    9100 2800
+	-1   0    0    1
+$EndComp
+Wire Wire Line
+	7850 3400 8300 3400
+Wire Wire Line
+	6750 3150 7750 3150
+Wire Wire Line
+	8300 3400 9100 3400
+Wire Wire Line
+	9100 3400 9100 3050
+Connection ~ 8300 3400
+$Comp
+L Device:C_Small C?
+U 1 1 5CEFE9A2
+P 9100 2950
+F 0 "C?" H 9192 2996 50  0000 L CNN
+F 1 "10PF" H 9192 2905 50  0000 L CNN
+F 2 "" H 9100 2950 50  0001 C CNN
+F 3 "~" H 9100 2950 50  0001 C CNN
+	1    9100 2950
+	1    0    0    -1
+$EndComp
+Wire Wire Line
+	9100 2850 9100 2800
+Connection ~ 9100 2800
+Wire Wire Line
+	8600 3100 8600 2950
+Wire Wire Line
+	8600 2900 8950 2900
+Wire Wire Line
+	8950 2900 8950 2800
+Connection ~ 8950 2800
+Wire Wire Line
+	8950 2800 9100 2800
+Wire Wire Line
+	8000 3100 8000 2950
+Wire Wire Line
+	8000 2950 8600 2950
+Connection ~ 8600 2950
+Wire Wire Line
+	8600 2950 8600 2900
+$Comp
+L Device:R_Small_US R?
+U 1 1 5CF06551
+P 7850 3100
+F 0 "R?" H 7700 3100 50  0000 L CNN
+F 1 "1M" H 7900 3100 50  0000 L CNN
+F 2 "" H 7850 3100 50  0001 C CNN
+F 3 "~" H 7850 3100 50  0001 C CNN
+	1    7850 3100
+	1    0    0    -1
+$EndComp
+Wire Wire Line
+	7750 3050 7750 3000
+Wire Wire Line
+	7750 3150 7750 3200
+Wire Wire Line
+	7750 3200 7850 3200
+Connection ~ 7850 3200
+Wire Wire Line
+	7850 3200 7850 3400
+Wire Wire Line
+	7850 3000 7750 3000
+Connection ~ 7850 3000
+Wire Wire Line
+	7850 2800 7850 3000
 $EndSCHEMATC

Commit message: annotated NRF905 shematic
Parts:
- U1: symbol CUSTOM:NRF905 -> GenLOCK-Drone-rescue:NRF905-CUSTOM
- gave numbers to parts that had none: 18
Changed lines of the file:
@@
 EESchema Schematic File Version 4
 LIBS:GenLOCK Drone-cache
-EELAYER 29 0
+EELAYER 26 0
 EELAYER END
 $Descr A4 11693 8268
@@
 $EndDescr
 $Comp
-L CUSTOM:NRF905 U1
+L GenLOCK-Drone-rescue:NRF905-CUSTOM U1
 U 1 1 5CECA706
 P 5950 2850
+AR Path="/5CECA706" Ref="U1"  Part="1"
+AR Path="/5CECA62C/5CECA706" Ref="U1"  Part="1"
 F 0 "U1" H 5950 3875 50  0000 C CNN
 F 1 "NRF905" H 5950 3784 50  0000 C CNN
@@
 Connection ~ 5150 3650
 $Comp
-L power:GNDREF #PWR?
+L power:GNDREF #PWR07
 U 1 1 5CECED0A
 P 5050 3650
-F 0 "#PWR?" H 5050 3400 50  0001 C CNN
+F 0 "#PWR07" H 5050 3400 50  0001 C CNN
 F 1 "GNDREF" V 5055 3522 50  0000 R CNN
 F 2 "" H 5050 3650 50  0001 C CNN
@@
 	5850 4350 5750 4350
 $Comp
-L power:+3.3V #PWR?
+L power:+3.3V #PWR08
 U 1 1 5CECF8C3
 P 5750 4350
-F 0 "#PWR?" H 5750 4200 50  0001 C CNN
+F 0 "#PWR08" H 5750 4200 50  0001 C CNN
 F 1 "+3.3V" V 5765 4478 50  0000 L CNN
 F 2 "" H 5750 4350 50  0001 C CNN
@@
 	5300 3900 5150 3900
 $Comp
-L Device:C_Small C?
+L Device:C_Small C8
 U 1 1 5CED4622
 P 5050 3900
-F 0 "C?" V 5150 3900 50  0000 C CNN
+F 0 "C8" V 5150 3900 50  0000 C CNN
 F 1 "10nF" V 4950 3900 50  0000 C CNN
 F 2 "" H 5050 3900 50  0001 C CNN
@@
 $EndComp
 $Comp
-L power:GNDREF #PWR?
+L power:GNDREF #PWR06
 U 1 1 5CED6115
 P 4950 3900
-F 0 "#PWR?" H 4950 3650 50  0001 C CNN
+F 0 "#PWR06" H 4950 3650 50  0001 C CNN
 F 1 "GNDREF" V 4955 3772 50  0000 R CNN
 F 2 "" H 4950 3900 50  0001 C CNN
@@
 	6600 3400 6750 3400
 $Comp
-L Device:R_Small_US R?
+L Device:R_Small_US R1
 U 1 1 5CED70DA
 P 6850 3400
-F 0 "R?" V 6645 3400 50  0000 C CNN
+F 0 "R1" V 6645 3400 50  0000 C CNN
 F 1 "22K" V 6736 3400 50  0000 C CNN
 F 2 "" H 6850 3400 50  0001 C CNN
@@
 	6950 3400 7100 3400
 $Comp
-L power:GNDREF #PWR?
+L power:GNDREF #PWR010
 U 1 1 5CED7B3B
 P 7100 3400
-F 0 "#PWR?" H 7100 3150 50  0001 C CNN
+F 0 "#PWR010" H 7100 3150 50  0001 C CNN
 F 1 "GNDREF" V 7105 3272 50  0000 R CNN
 F 2 "" H 7100 3400 50  0001 C CNN
@@
 	4350 3750 4350 3850
 $Comp
-L Device:C_Small C?
+L Device:C_Small C4
 U 1 1 5CED52A1
 P 4350 3950
-F 0 "C?" V 4450 3950 50  0000 C CNN
+F 0 "C4" V 4450 3950 50  0000 C CNN
 F 1 "3.3nF" V 4250 3950 50  0000 C CNN
 F 2 "" H 4350 3950 50  0001 C CNN
@@
 $EndComp
 $Comp
-L power:GNDREF #PWR?
+L power:GNDREF #PWR03
 U 1 1 5CED5DBC
 P 4350 4050
-F 0 "#PWR?" H 4350 3800 50  0001 C CNN
+F 0 "#PWR03" H 4350 3800 50  0001 C CNN
 F 1 "GNDREF" V 4355 3922 50  0000 R CNN
 F 2 "" H 4350 4050 50  0001 C CNN
@@
 	4850 1750 4850 2050
 $Comp
-L Device:C_Small C?
+L Device:C_Small C6
 U 1 1 5CED9A7D
 P 4400 2100
-F 0 "C?" H 4492 2146 50  0000 L CNN
+F 0 "C6" H 4492 2146 50  0000 L CNN
 F 1 "0F" H 4492 2055 50  0000 L CNN
 F 2 "" H 4400 2100 50  0001 C CNN
@@
 	4400 2450 4850 2450
 $Comp
-L Device:C_Small C?
+L Device:C_Small C7
 U 1 1 5CEDBFEF
 P 4400 2550
-F 0 "C?" H 4492 2596 50  0000 L CNN
+F 0 "C7" H 4492 2596 50  0000 L CNN
 F 1 "18PF" H 4492 2505 50  0000 L CNN
 F 2 "" H 4400 2550 50  0001 C CNN
@@
 $EndComp
 $Comp
-L Device:C_Small C?
+L Device:C_Small C5
 U 1 1 5CEDC357
 P 4400 1650
-F 0 "C?" H 4492 1696 50  0000 L CNN
+F 0 "C5" H 4492 1696 50  0000 L CNN
 F 1 "18PF" H 4492 1605 50  0000 L CNN
 F 2 "" H 4400 1650 50  0001 C CNN
@@
 $EndComp
 $Comp
-L power:GNDREF #PWR?
+L power:GNDREF #PWR05
 U 1 1 5CEDC733
 P 4400 2650
-F 0 "#PWR?" H 4400 2400 50  0001 C CNN
+F 0 "#PWR05" H 4400 2400 50  0001 C CNN
 F 1 "GNDREF" H 4405 2477 50  0000 C CNN
 F 2 "" H 4400 2650 50  0001 C CNN
@@
 $EndComp
 $Comp
-L power:GNDREF #PWR?
+L power:GNDREF #PWR04
 U 1 1 5CEDC9CC
 P 4400 1550
-F 0 "#PWR?" H 4400 1300 50  0001 C CNN
+F 0 "#PWR04" H 4400 1300 50  0001 C CNN
 F 1 "GNDREF" H 4405 1377 50  0000 C CNN
 F 2 "" H 4400 1550 50  0001 C CNN
@@
 $EndComp
 $Comp
-L pspice:INDUCTOR L?
+L pspice:INDUCTOR L3
 U 1 1 5CEDCDC7
 P 3950 2100
-F 0 "L?" V 3904 2178 50  0000 L CNN
+F 0 "L3" V 3904 2178 50  0000 L CNN
 F 1 "12nH" V 3995 2178 50  0000 L CNN
 F 2 "" H 3950 2100 50  0001 C CNN
@@
 Connection ~ 3950 1750
 $Comp
-L pspice:INDUCTOR L?
+L pspice:INDUCTOR L1
 U 1 1 5CEDE77F
 P 3600 1750
-F 0 "L?" H 3450 1850 50  0000 C CNN
+F 0 "L1" H 3450 1850 50  0000 C CNN
 F 1 "39nH" H 3700 1850 50  0000 C CNN
 F 2 "" H 3600 1750 50  0001 C CNN
@@
 Connection ~ 4350 3750
 $Comp
-L Device:C_Small C?
+L Device:C_Small C3
 U 1 1 5CEE10EB
 P 3200 1750
-F 0 "C?" V 2971 1750 50  0000 C CNN
+F 0 "C3" V 2971 1750 50  0000 C CNN
 F 1 "180PF" V 3062 1750 50  0000 C CNN
 F 2 "" H 3200 1750 50  0001 C CNN
@@
 	3100 1750 3000 1750
 $Comp
-L power:GNDREF #PWR?
+L power:GNDREF #PWR01
 U 1 1 5CEE2B51
 P 3000 1750
-F 0 "#PWR?" H 3000 1500 50  0001 C CNN
+F 0 "#PWR01" H 3000 1500 50  0001 C CNN
 F 1 "GNDREF" V 3005 1622 50  0000 R CNN
 F 2 "" H 3000 1750 50  0001 C CNN
@@
 $EndComp
 $Comp
-L pspice:INDUCTOR L?
+L pspice:INDUCTOR L2
 U 1 1 5CEE2D59
 P 3600 2450
-F 0 "L?" H 3450 2550 50  0000 C CNN
+F 0 "L2" H 3450 2550 50  0000 C CNN
 F 1 "39nH" H 3700 2550 50  0000 C CNN
 F 2 "" H 3600 2450 50  0001 C CNN
@@
 Connection ~ 3950 2450
 $Comp
-L Device:C_Small C?
+L Device:C_Small C2
 U 1 1 5CEE5F1E
 P 3150 2450
-F 0 "C?" V 2921 2450 50  0000 C CNN
+F 0 "C2" V 2921 2450 50  0000 C CNN
 F 1 "6.8PF" V 3012 2450 50  0000 C CNN
 F 2 "" H 3150 2450 50  0001 C CNN
@@
 	3000 2450 2950 2450
 $Comp
-L Device:C_Small C?
+L Device:C_Small C1
 U 1 1 5CEEA35A
 P 3000 2600
-F 0 "C?" H 3092 2646 50  0000 L CNN
+F 0 "C1" H 3092 2646 50  0000 L CNN
 F 1 "0F" H 3092 2555 50  0000 L CNN
 F 2 "" H 3000 2600 50  0001 C CNN
@@
 $EndComp
 $Comp
-L power:GNDREF #PWR?
+L power:GNDREF #PWR02
 U 1 1 5CEEA8A2
 P 3000 2700
-F 0 "#PWR?" H 3000 2450 50  0001 C CNN
+F 0 "#PWR02" H 3000 2450 50  0001 C CNN
 F 1 "GNDREF" H 3005 2527 50  0000 C CNN
 F 2 "" H 3000 2700 50  0001 C CNN
@@
 $EndComp
 $Comp
-L Device:Antenna AE?
+L Device:Antenna AE1
 U 1 1 5CEEB254
 P 2750 2450
-F 0 "AE?" V 2967 2393 50  0000 C CNN
+F 0 "AE1" V 2967 2393 50  0000 C CNN
 F 1 "Antenna" V 2876 2393 50  0000 C CNN
 F 2 "" H 2750 2450 50  0001 C CNN
@@
 Connection ~ 6050 4350
 $Comp
-L Device:C_Small C?
+L Device:C_Small C9
 U 1 1 5CEDE401
 P 6250 4350
-F 0 "C?" V 6400 4350 50  0000 C CNN
+F 0 "C9" V 6400 4350 50  0000 C CNN
 F 1 "33PF" V 6112 4350 50  0000 C CNN
 F 2 "" H 6250 4350 50  0001 C CNN
@@
 $EndComp
 $Comp
-L power:GNDREF #PWR?
+L power:GNDREF #PWR09
 U 1 1 5CEDF64B
 P 6350 4350
-F 0 "#PWR?" H 6350 4100 50  0001 C CNN
+F 0 "#PWR09" H 6350 4100 50  0001 C CNN
 F 1 "GNDREF" V 6355 4222 50  0000 R CNN
 F 2 "" H 6350 4350 50  0001 C CNN
@@
 	6700 3150 6700 3050
 $Comp
-L Oscillator:XO32 X?
+L Oscillator:XO32 X1
 U 1 1 5CEF225C
 P 8300 3100
-F 0 "X?" V 8254 3444 50  0000 L CNN
+F 0 "X1" V 8254 3444 50  0000 L CNN
 F 1 "XO32" V 8345 3444 50  0000 L CNN
 F 2 "Oscillator:Oscillator_SMD_EuroQuartz_XO32-4Pin_3.2x2.5mm" H 9000 2750 50  0001 C CNN
@@
 Connection ~ 8300 2800
 $Comp
-L Device:C_Small C?
+L Device:C_Small C10
 U 1 1 5CEF7465
 P 8750 2800
-F 0 "C?" V 8521 2800 50  0000 C CNN
+F 0 "C10" V 8521 2800 50  0000 C CNN
 F 1 "10PF" V 8612 2800 50  0000 C CNN
 F 2 "" H 8750 2800 50  0001 C CNN
@@
 	8850 2800 8950 2800
 $Comp
-L power:GNDREF #PWR?
+L power:GNDREF #PWR011
 U 1 1 5CEF9ACB
 P 9100 2800
-F 0 "#PWR?" H 9100 2550 50  0001 C CNN
+F 0 "#PWR011" H 9100 2550 50  0001 C CNN
 F 1 "GNDREF" H 9105 2627 50  0000 C CNN
 F 2 "" H 9100 2800 50  0001 C CNN
@@
 Connection ~ 8300 3400
 $Comp
-L Device:C_Small C?
+L Device:C_Small C11
 U 1 1 5CEFE9A2
 P 9100 2950
-F 0 "C?" H 9192 2996 50  0000 L CNN
+F 0 "C11" H 9192 2996 50  0000 L CNN
 F 1 "10PF" H 9192 2905 50  0000 L CNN
 F 2 "" H 9100 2950 50  0001 C CNN
@@
 	8600 2950 8600 2900
 $Comp
-L Device:R_Small_US R?
+L Device:R_Small_US R2
 U 1 1 5CF06551
 P 7850 3100
-F 0 "R?" H 7700 3100 50  0000 L CNN
+F 0 "R2" H 7700 3100 50  0000 L CNN
 F 1 "1M" H 7900 3100 50  0000 L CNN
 F 2 "" H 7850 3100 50  0001 C CNN
